Commit message: Mapping project. First commit. Josh Chen 6/14/2020

File: catkin_ws/src/my_robot/urdf/my_robot.xacro (robot description, xacro)
@@ -176,4 +176,11 @@
     <axis xyz="0 1 0" rpy="0 0 0"/>
   </joint>
+  <joint type="fixed" name="camera_optical_joint">
+    <origin xyz="0 0 0" rpy="-1.5707 0 -1.5707"/>
+    <child link="camera_link_optical"/>
+    <parent link="camera"/>
+  </joint>
+  <link name="camera_link_optical">
+  </link>
   <gazebo reference="left_wheel">
     <material>Gazebo/SkyBlue</material>
